Commit message: changed names of links and joints in urdf

File: capsules/fb_kairos_ur5e_oem_capsules.urdf (robot description, URDF)
Before this commit: robot rb_kairos_ur10e, 33 links, 32 joints
Links:
- removed link rb_kairos_back_left_wheel_link
- removed link rb_kairos_back_right_wheel_link
- removed link rb_kairos_base_chapa
- removed link rb_kairos_base_docking_contact
- removed link rb_kairos_base_footprint
- removed link rb_kairos_base_link
- removed link rb_kairos_base_logo_front
- removed link rb_kairos_base_logo_left
- removed link rb_kairos_base_logo_rear
- removed link rb_kairos_base_logo_right
- removed link rb_kairos_front_laser_base_link
- removed link rb_kairos_front_laser_link
- removed link rb_kairos_front_left_wheel_link
- removed link rb_kairos_front_rgbd_camera_depth_frame
- removed link rb_kairos_front_rgbd_camera_depth_optical_frame
- removed link rb_kairos_front_rgbd_camera_link
- removed link rb_kairos_front_rgbd_camera_rgb_frame
- removed link rb_kairos_front_rgbd_camera_rgb_optical_frame
- removed link rb_kairos_front_right_wheel_link
- removed link rb_kairos_imu_link
- removed link rb_kairos_rear_laser_base_link
- removed link rb_kairos_rear_laser_link
- removed link rb_kairos_ur16e_EE
- removed link rb_kairos_ur16e_base
- removed link rb_kairos_ur16e_base_link
- removed link rb_kairos_ur16e_flange
- removed link rb_kairos_ur16e_forearm_link
- removed link rb_kairos_ur16e_shoulder_link
- removed link rb_kairos_ur16e_upper_arm_link
- removed link rb_kairos_ur16e_wrist_1_link
- removed link rb_kairos_ur16e_wrist_2_link
- removed link rb_kairos_ur16e_wrist_3_link
- added link rbkairos_back_left_wheel_link, mass 6.5; collision cylinder length=0.087 radius=0.127; visual mesh filename=package://hrii_robotnik_description/meshes/wheels/omni_whee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
- added link rbkairos_back_right_wheel_link, mass 6.5; collision cylinder length=0.087 radius=0.127; visual mesh filename=package://hrii_robotnik_description/meshes/wheels/omni_whee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
- added link rbkairos_base_chapa; visual mesh filename=package://hrii_robotnik_description/meshes/bases/xls/summit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
- added link rbkairos_base_docking_contact
- added link rbkairos_base_footprint; visual box size=0.001 0.001 0.001
- added link rbkairos_base_link, mass 125.0; collision cylinder length=0.2105700249070154 radius=0.474306; visual mesh filename=package://hrii_robotnik_description/meshes/bases/xls/summit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
- added link rbkairos_base_logo_front; visual mesh filename=package://hrii_robotnik_description/meshes/bases/xls/robotn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
- added link rbkairos_base_logo_left; visual mesh filename=package://hrii_robotnik_description/meshes/bases/xls/robotn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
- added link rbkairos_base_logo_rear; visual mesh filename=package://hrii_robotnik_description/meshes/bases/xls/robotn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
- added link rbkairos_base_logo_right; visual mesh filename=package://hrii_robotnik_description/meshes/bases/xls/robotn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
- added link rbkairos_front_laser_base_link, mass 0.13; collision box size=0.01 0.01 0.01; visual mesh filename=package://robotnik_sensors/meshes/hokuyo_ust_10lx.dae
- added link rbkairos_front_laser_link
- added link rbkairos_front_left_wheel_link, mass 6.5; collision cylinder length=0.087 radius=0.127; visual mesh filename=package://hrii_robotnik_description/meshes/wheels/omni_whee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
- added link rbkairos_front_rgbd_camera_depth_frame, mass 0.001
- added link rbkairos_front_rgbd_camera_depth_optical_frame, mass 0.001
- added link rbkairos_front_rgbd_camera_link, mass 0.001
- added link rbkairos_front_rgbd_camera_rgb_frame, mass 0.297
- added link rbkairos_front_rgbd_camera_rgb_optical_frame, mass 0.001
- added link rbkairos_front_right_wheel_link, mass 6.5; collision cylinder length=0.087 radius=0.127; visual mesh filename=package://hrii_robotnik_description/meshes/wheels/omni_whee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
- added link rbkairos_imu_link, mass 0.05; collision box size=0.001 0.001 0.001; visual box size=0.001 0.001 0.001
- added link rbkairos_rear_laser_base_link, mass 0.13; collision box size=0.01 0.01 0.01; visual mesh filename=package://robotnik_sensors/meshes/hokuyo_ust_10lx.dae
- added link rbkairos_rear_laser_link
- added link rbkairos_ur5e_EE
- added link rbkairos_ur5e_base
- added link rbkairos_ur5e_base_link, mass 4.0; visual mesh filename=package://hrii_universal_robots_description/meshes/ur5e/vis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
- added link rbkairos_ur5e_flange, mass 0.1879
- added link rbkairos_ur5e_forearm_link, mass 2.275; collision cylinder length=0.3587816604615533 radius=0.073314; visual mesh filename=package://hrii_universal_robots_description/meshes/ur5e/vis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
- added link rbkairos_ur5e_shoulder_link, mass 3.7; collision cylinder length=0.014226880885683055 radius=0.0832319; visual mesh filename=package://hrii_universal_robots_description/meshes/ur5e/vis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
- added link rbkairos_ur5e_upper_arm_link, mass 8.393; collision cylinder length=0.44747021827210387 radius=0.110215; visual mesh filename=package://hrii_universal_robots_description/meshes/ur5e/vis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
- added link rbkairos_ur5e_wrist_1_link, mass 1.219; collision cylinder length=0.024887588224355536 radius=0.0727752; visual mesh filename=package://hrii_universal_robots_description/meshes/ur5e/vis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
- added link rbkairos_ur5e_wrist_2_link, mass 1.219; collision cylinder length=0.026628540549890157 radius=0.0644024; visual mesh filename=package://hrii_universal_robots_description/meshes/ur5e/vis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
- added link rbkairos_ur5e_wrist_3_link, mass 0.1879; collision cylinder length=0.004160703963552799 radius=0.0494953; visual mesh filename=package://hrii_universal_robots_description/meshes/ur5e/vis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
Joints:
- removed joint rb_kairos_back_left_wheel_joint
- removed joint rb_kairos_back_right_wheel_joint
- removed joint rb_kairos_base_docking_joint
- removed joint rb_kairos_base_footprint_joint
- removed joint rb_kairos_base_logo_front_joint
- removed joint rb_kairos_base_logo_left_joint
- removed joint rb_kairos_base_logo_rear_joint
- removed joint rb_kairos_base_logo_right_joint
- removed joint rb_kairos_base_tapa_joint
- removed joint rb_kairos_front_laser_base_joint
- removed joint rb_kairos_front_laser_joint
- removed joint rb_kairos_front_left_wheel_joint
- removed joint rb_kairos_front_rgbd_camera_depth_joint
- removed joint rb_kairos_front_rgbd_camera_depth_optical_joint
- removed joint rb_kairos_front_rgbd_camera_joint
- removed joint rb_kairos_front_rgbd_camera_rgb_joint
- removed joint rb_kairos_front_rgbd_camera_rgb_optical_joint
- removed joint rb_kairos_front_right_wheel_joint
- removed joint rb_kairos_imu_joint
- removed joint rb_kairos_joint_ur16e_link0_base_footprint
- removed joint rb_kairos_rear_laser_base_joint
- removed joint rb_kairos_rear_laser_joint
- removed joint rb_kairos_ur16e_base_link-base_fixed_joint
- removed joint rb_kairos_ur16e_elbow_joint
- removed joint rb_kairos_ur16e_joint_EE
- removed joint rb_kairos_ur16e_shoulder_lift_joint
- removed joint rb_kairos_ur16e_shoulder_pan_joint
- removed joint rb_kairos_ur16e_wrist_1_joint
- removed joint rb_kairos_ur16e_wrist_2_joint
- removed joint rb_kairos_ur16e_wrist_3_joint
- removed joint rb_kairos_ur16e_wrist_3_link_flange_fixed_joint
- added joint rbkairos_back_left_wheel_joint: type continuous, parent rbkairos_base_link, child rbkairos_back_left_wheel_link, origin xyz=-0.21528 0.269 0.0 rpy=0.0 0.0 0.0, axis 0.0 1.0 0.0, limit lower=0 upper=0 effort=100.0 velocity=100.0
- added joint rbkairos_back_right_wheel_joint: type continuous, parent rbkairos_base_link, child rbkairos_back_right_wheel_link, origin xyz=-0.21528 -0.269 0.0 rpy=0.0 0.0 0.0, axis 0.0 1.0 0.0, limit lower=0 upper=0 effort=100.0 velocity=100.0
- added joint rbkairos_base_docking_joint: type fixed, parent rbkairos_base_link, child rbkairos_base_docking_contact, origin xyz=0.35 0.0 0.09 rpy=0.0 0.0 0.0
- added joint rbkairos_base_footprint_joint: type fixed, parent rbkairos_base_footprint, child rbkairos_base_link, origin xyz=0.0 0.0 0.127 rpy=0.0 0.0 0.0
- added joint rbkairos_base_logo_front_joint: type fixed, parent rbkairos_base_link, child rbkairos_base_logo_front, origin xyz=0.345 0.0 0.0 rpy=0.0 0.0 -1.5707963267948966
- added joint rbkairos_base_logo_left_joint: type fixed, parent rbkairos_base_link, child rbkairos_base_logo_left, origin xyz=0.0 0.28931 0.29062 rpy=0.0 0.0 0.0
- added joint rbkairos_base_logo_rear_joint: type fixed, parent rbkairos_base_link, child rbkairos_base_logo_rear, origin xyz=-0.345 0.0 0.0 rpy=0.0 0.0 1.5707963267948966
- added joint rbkairos_base_logo_right_joint: type fixed, parent rbkairos_base_link, child rbkairos_base_logo_right, origin xyz=0.0 -0.28931 0.29062 rpy=0.0 0.0 3.141592653589793
- added joint rbkairos_base_tapa_joint: type fixed, parent rbkairos_base_link, child rbkairos_base_chapa, origin xyz=0.0 0.0 0.38062 rpy=0.0 0.0 0.0
- added joint rbkairos_front_laser_base_joint: type fixed, parent rbkairos_base_link, child rbkairos_front_laser_base_link, origin xyz=0.28783 -0.2224 0.22365 rpy=0.0 3.14159 2.3561924999999997
- added joint rbkairos_front_laser_joint: type fixed, parent rbkairos_front_laser_base_link, child rbkairos_front_laser_link, origin xyz=0.0 0.0 0.0474 rpy=0.0 0.0 0.0
- added joint rbkairos_front_left_wheel_joint: type continuous, parent rbkairos_base_link, child rbkairos_front_left_wheel_link, origin xyz=0.21528 0.269 0.0 rpy=0.0 0.0 0.0, axis 0.0 1.0 0.0, limit lower=0 upper=0 effort=100.0 velocity=100.0
- added joint rbkairos_front_rgbd_camera_depth_joint: type fixed, parent rbkairos_front_rgbd_camera_link, child rbkairos_front_rgbd_camera_depth_frame, origin xyz=0.0 0.0375 0.015 rpy=0.0 0.0 0.0
- added joint rbkairos_front_rgbd_camera_depth_optical_joint: type fixed, parent rbkairos_front_rgbd_camera_depth_frame, child rbkairos_front_rgbd_camera_depth_optical_frame, origin xyz=0.0 0.0 0.0 rpy=-1.5707963267948966 0.0 -1.5707963267948966
- added joint rbkairos_front_rgbd_camera_joint: type fixed, parent rbkairos_base_link, child rbkairos_front_rgbd_camera_link, origin xyz=0.3585 0.0 0.28062 rpy=0.0 0.0 0.0
- added joint rbkairos_front_rgbd_camera_rgb_joint: type fixed, parent rbkairos_front_rgbd_camera_link, child rbkairos_front_rgbd_camera_rgb_frame, origin xyz=0.0 0.0125 0.015 rpy=0.0 0.0 0.0
- added joint rbkairos_front_rgbd_camera_rgb_optical_joint: type fixed, parent rbkairos_front_rgbd_camera_rgb_frame, child rbkairos_front_rgbd_camera_rgb_optical_frame, origin xyz=0.0 0.0 0.0 rpy=-1.5707963267948966 0.0 -1.5707963267948966
- added joint rbkairos_front_right_wheel_joint: type continuous, parent rbkairos_base_link, child rbkairos_front_right_wheel_link, origin xyz=0.21528 -0.269 0.0 rpy=0.0 0.0 0.0, axis 0.0 1.0 0.0, limit lower=0 upper=0 effort=100.0 velocity=100.0
- added joint rbkairos_imu_joint: type fixed, parent rbkairos_base_link, child rbkairos_imu_link, origin xyz=0.127 -0.129 0.212 rpy=0.0 0.0 0.0, axis 1.0 0.0 0.0
- added joint rbkairos_joint_ur5e_link0_base_footprint: type fixed, parent rbkairos_base_chapa, child rbkairos_ur5e_base_link, origin xyz=0.15887 0.0 0.18062 rpy=0.0 0.0 0.0
- added joint rbkairos_rear_laser_base_joint: type fixed, parent rbkairos_base_link, child rbkairos_rear_laser_base_link, origin xyz=-0.28783 0.2224 0.22365 rpy=0.0 3.14159 -0.7853975
- added joint rbkairos_rear_laser_joint: type fixed, parent rbkairos_rear_laser_base_link, child rbkairos_rear_laser_link, origin xyz=0.0 0.0 0.0474 rpy=0.0 0.0 0.0
- added joint rbkairos_ur5e_base_link-base_fixed_joint: type fixed, parent rbkairos_ur5e_base_link, child rbkairos_ur5e_base, origin xyz=0.0 0.0 0.0 rpy=0.0 0.0 -3.14159
- added joint rbkairos_ur5e_elbow_joint: type continuous, parent rbkairos_ur5e_upper_arm_link, child rbkairos_ur5e_forearm_link, origin xyz=-0.425 0.0 0.0 rpy=0.0 0.0 0.0, axis 0.0 0.0 1.0, limit lower=-6.28318 upper=6.28318 effort=150.0 velocity=3.15
- added joint rbkairos_ur5e_joint_EE: type fixed, parent rbkairos_ur5e_flange, child rbkairos_ur5e_EE, origin xyz=0.0 0.0 0.0 rpy=0.0 0.0 0.0, axis 0.0 0.0 0.0
- added joint rbkairos_ur5e_shoulder_lift_joint: type continuous, parent rbkairos_ur5e_shoulder_link, child rbkairos_ur5e_upper_arm_link, origin xyz=0.0 0.0 0.0 rpy=1.570795 0.0 0.0, axis 0.0 0.0 1.0, limit lower=-6.28318 upper=6.28318 effort=150.0 velocity=3.15
- added joint rbkairos_ur5e_shoulder_pan_joint: type continuous, parent rbkairos_ur5e_base_link, child rbkairos_ur5e_shoulder_link, origin xyz=0.0 0.0 0.1625 rpy=0.0 0.0 3.14159, axis 0.0 0.0 1.0, limit lower=-6.28318 upper=6.28318 effort=150.0 velocity=3.15
- added joint rbkairos_ur5e_wrist_1_joint: type continuous, parent rbkairos_ur5e_forearm_link, child rbkairos_ur5e_wrist_1_link, origin xyz=-0.3922 0.0 0.1333 rpy=0.0 0.0 0.0, axis 0.0 0.0 1.0, limit lower=-6.28318 upper=6.28318 effort=28.0 velocity=6.28
- added joint rbkairos_ur5e_wrist_2_joint: type continuous, parent rbkairos_ur5e_wrist_1_link, child rbkairos_ur5e_wrist_2_link, origin xyz=0.0 -0.0997 0.0 rpy=1.570795 0.0 0.0, axis 0.0 0.0 1.0, limit lower=-6.28318 upper=6.28318 effort=28.0 velocity=3.2
- added joint rbkairos_ur5e_wrist_3_joint: type continuous, parent rbkairos_ur5e_wrist_2_link, child rbkairos_ur5e_wrist_3_link, origin xyz=0.0 0.0996 0.0 rpy=1.570795 3.14159 3.14159, axis 0.0 0.0 1.0, limit lower=-6.28318 upper=6.28318 effort=28.0 velocity=6.28
- added joint rbkairos_ur5e_wrist_3_link_flange_fixed_joint: type fixed, parent rbkairos_ur5e_wrist_3_link, child rbkairos_ur5e_flange, origin xyz=0.0 0.0 0.0 rpy=0.0 0.0 0.0
- joint reference: child rb_kairos_base_footprint -> rbkairos_base_footprint
